File: ControllerHW/DuploTrainController/DuploTrainController.kicad_sch (KiCad schematic)
At the start: 0 parts

Commit message: Traincontroller Buttons are working after Logging was modified to  log without semaphor
Parts:
- added J1: Taster Kabel (rot), symbol Connector:Conn_01x03_Pin
- added J2: Taster Kabel (gelb), symbol Connector:Conn_01x02_Pin
- added J3: Fahrtregler Kabel (gelb rot), symbol Connector:Conn_01x02_Pin
- added RV1: Speed, symbol Device:R_Potentiometer
- added SW1: Not Aus (rot), symbol Switch:SW_Push
- added SW2: Sound Cycle (gelb), symbol Switch:SW_Push
- added SW3: LED Cycle (weiß), symbol Switch:SW_Push
- added SW4: Water (blau), symbol Switch:SW_Push
- added U1: ESP32-WROOM-32, RF_Module:ESP32-WROOM-32, symbol RF_Module:ESP32-WROOM-32
Connections:
- new net: J1.3 (Pin_3), RV1.1, SW1.2, SW2.1, SW3.1, SW4.2
- new net: J3.1 (Pin_1), RV1.2
- new net: J3.2 (Pin_2), RV1.3
- new net: J1.1 (Pin_1), SW1.1
- new net: J1.2 (Pin_2), SW4.1
- new net: J2.1 (Pin_1), SW3.2
- new net: J2.2 (Pin_2), SW2.2
- new net +3V3: U1.2 (VDD)
- new net Fahrstufe: U1.23 (IO15)
- new net GND: U1.1 (GND), U1.15 (GND), U1.38 (GND), U1.39 (GND)
- new net Geräusasuwahl: U1.12 (IO27)
- new net Lichtauswahl: U1.11 (IO26)
- new net Not_Aus: U1.13 (IO14)
- new net Wasseraufnahme: U1.10 (IO25)
Other:
- note added: "Fahrpult für einen Duplo Zug - aktuell keine LED für Power Anzeige da Batteriebetrieb - Taster sollten über kleines PCB verbunden werden (Abstand 41mm)"
- note added: "braune Ader"
- note added: "rote Ader"
- note added: "schwarze Ader"
